File: pcb/faboy/faboy.sch (EAGLE design)
At the start: 53 parts, among them J1 USB-MICROBREDUCED_PASTE, U1 MAX1595UMAX, U2 MCP73831, Y1 16MHZ

Commit message: add games
Parts:
- R10, R11, R5, R6, R9: value 330 -> 820
Changed lines of the file:
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@@
 <part name="LED1" library="led" deviceset="LED" device="SML0805"/>
 <part name="LED2" library="led" deviceset="LED" device="SML0805"/>
-<part name="R5" library="resistor" deviceset="R-EU_" device="R0805" value="330"/>
-<part name="R6" library="resistor" deviceset="R-EU_" device="R0805" value="330"/>
+<part name="R5" library="resistor" deviceset="R-EU_" device="R0805" value="820"/>
+<part name="R6" library="resistor" deviceset="R-EU_" device="R0805" value="820"/>
 <part name="P+3" library="supply1" deviceset="VCC" device=""/>
 <part name="C10" library="resistor" deviceset="C-EU" device="C0805K" value="1uF"/>
@@
 <part name="C16" library="resistor" deviceset="C-EU" device="C0805K" value="4.7uF"/>
 <part name="GND24" library="supply1" deviceset="GND" device=""/>
-<part name="R9" library="resistor" deviceset="R-EU_" device="R0805" value="330"/>
-<part name="R10" library="resistor" deviceset="R-EU_" device="R0805" value="330"/>
-<part name="R11" library="resistor" deviceset="R-EU_" device="R0805" value="330"/>
+<part name="R9" library="resistor" deviceset="R-EU_" device="R0805" value="820"/>
+<part name="R10" library="resistor" deviceset="R-EU_" device="R0805" value="820"/>
+<part name="R11" library="resistor" deviceset="R-EU_" device="R0805" value="820"/>
 <part name="U$7" library="SparkFun-LED" deviceset="LED-RGB-P-LCC-4" device=""/>
 <part name="P+4" library="supply1" deviceset="VCC" device=""/>
