File: pcb/faboy_ble/faboy_ble.sch (EAGLE design)
At the start: 52 parts, among them J1 USB-MICROBREDUCED_PASTE, U1 MAX1595UMAX, U2 MCP73831

Commit message: pcb ble routing
Parts:
- removed C11: 0.47uF, resistor:C-EUC0805K
- removed C12, C13: 2.2uF, resistor:C-EUC0805K
- removed C8: 1uF, resistor:C-EUC0805K
- removed C9: 0.1uF, resistor:C-EUC0805K
- removed F1: 500mA, adafruit:PTCFUSE-1812
- removed J2: (no value), SparkFun-Connectors:M06SMD-FEMALE-V2
- removed SJ1: direct power, jumper:SJ
- removed U3: (no value), BMD-200-Eagle:BMD-200
- added IC1: FT230XS, ftdichip:FT230XS
- added R13: ferrite, resistor:R-EU_R0805
- added U$2: WT51822-02, Wireless_Tag:WT51822-02
- added U$9: MICROSD, adafruit:MICROSD
- C10: value 1uF -> 2.2uF
- C7: value 1uF -> 0.1uF
- S1, S2, S3, S4, S6, S7: value SWITCH-MOMENTARY-2SMD-REDUNDANT -> SWITCH-MOMENTARY-2SMD-4; device SparkFun-Electromechanical:SWITCH-MOMENTARY-2SMD-REDUNDANT -> SparkFun-Electromechanical:SWITCH-MOMENTARY-2SMD-4
- U1: value MAX1595UMAX -> 3.3V/150mA; device maxim:MAX1595UMAX -> SparkFun-PowerIC:V_REG_MIC52053.3V
Connections:
- removed net N$15: C11.1, U1.CXN
- removed net N$16: C11.2, U1.CXP
- removed net N$20: C16.2
- removed net N$26: SG1.2
- new net 3V3: C7.1, IC1.!RESET, IC1.3V3OUT, IC1.VCCIO, LED1.A, LED2.A
- new net CTS: IC1.!CTS, U$2.P0.13
- new net N$11: C16.1, SG1.2
- new net RTS: IC1.!RTS, U$2.P0.15
- new net RX: IC1.RXD, U$2.P0.14
- new net TX: IC1.TXD, U$2.P0.16
- net A: now also U$2.P0.29
- net B: now also U$2.P0.28
- net BLUE: now also U$2.P0.24
- net CS: now also U$2.P0.05
- net D+: now also IC1.USBDP
- net D-: now also IC1.USBDM
- net DC: now also U$2.P0.03
- net DOWN: now also S4.1, U$2.P0.10; no longer S1.1
- net GND: now also C10.2, C7.2, IC1.GND, IC1.GND@1, U$2.GND@1, U$2.GND@2, U$2.GND@3, U$2.GND@4, U$2.GND@5; no longer C10.1, C12.2, C13.2, C7.1, C8.2, C9.2, J2.1, U1.PGND
- net GREEN: now also U$2.P0.23
- net LED_RX: now also IC1.CBUS0, R5.2; no longer R6.2
- net LED_TX: now also IC1.CBUS1, R6.2; no longer R5.2
- net LEFT: now also S3.1, U$2.P0.11; no longer S2.1
- net MISO: now also U$2.P0.00; no longer J2.3
- net MOSI: now also U$2.P0.01; no longer J2.4
- net N$10: now also C16.2, U$2.P0.27; no longer C12.1, S5.S, SJ1.1, U1.!SHDN, U1.IN
- net N$21: now also U$2.P0.26; no longer C16.1
- net N$9: now also S5.O, U1.EN, U1.IN; no longer C7.2
- net OLED_RST: now also U$2.P0.04
- net RED: now also U$2.P0.25
- net RIGHT: now also S2.1, U$2.P0.09; no longer S3.1
- net RST: no longer J2.2
- net SCLK: now also U$2.P0.02; no longer J2.5
- net UP: now also S1.1, U$2.P0.08; no longer S4.1
- net VBAT: now also U$2.P0.20
- net VBUS: now also R13.2; no longer F1.1
- net VCC: now also C10.1, U$2.VCC; no longer C13.1, J2.6, LED1.A, LED2.A, SJ1.2, U1.AOUT
- net VIN: now also IC1.VCC, R13.1; no longer C10.2, C8.1, C9.1, F1.2
Other:
- moved on the sheet: BAT1, C10, C14, C15, C16, C7, LED1, LED2, LED3, R12, R5, R6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

Commit message: ble pcb design done
Parts:
- added C8: 22nF, resistor:C-EUC0805K
- added J2: CORTEX_DEBUGSMD, SparkFun-Connectors:CORTEX_DEBUGSMD
- added R14: 2.2M, resistor:R-EU_R0805
- added SJ1: conf_2, jumper:SJ
- added TP1, TP2, TP3, TP4, TP5: TPB1,27, testpad:TPB1,27
- R2: value 10k -> 10M
- SJ3: value direct path -> conf_1
Connections:
- net CS renamed CS_OLED
- new net CS_SD: U$2.P0.00, U$9.CS
- new net MES_BAT: C8.1, R14.1, R2.2, TP1.TP, U$2.P0.20
- new net SD_DETECT: U$2.P0.07, U$9.CARD_DETECT
- new net SWDCLK: J2.SWDCLK/TCK, U$2.SWDIO
- new net SWDIO: J2.SWDIO/TMS, U$2.SWDCLK
- new net VSS: U$9.GND, U$9.GND1, U$9.VSS
- net 3V3: now also SJ3.1
- net GND: now also C8.2, J2.GND@3, J2.GND@5, J2.GNDDTCT, J2.NRESET, R14.2, TP5.TP, U$2.ANTEN
- net MISO: now also U$2.P0.06, U$9.DATA_OUT; no longer U$2.P0.00
- net MOSI: now also U$9.DATA_IN
- net N$9: now also SJ1.1
- net RST: now also U$2.P0.21; no longer R2.1
- net SCLK: now also U$9.SCLK
- net VBAT: now also R2.1, SJ3.3, TP3.TP; no longer SJ3.1, U$2.P0.20
- net VCC: now also J2.VCC, SJ1.2, TP4.TP, U$9.VDD; no longer R2.2
- net VIN: now also TP2.TP; no longer SJ3.3
Other:
- moved on the sheet: R2, S5, S8, SJ3
